File: my_power_supply.kicad_sch (KiCad schematic)
At the start: 61 parts, among them J1 USB_C_Receptacle_USB2.0_16P, J2 USB_C_Receptacle_PowerOnly_6P, J3 USB_C_Receptacle_PowerOnly_6P, Q1 AONR21307, SW1 SW_SPST, SW2 SW_SPST, U2 TPS54560BDDA, U3 HUSB238, U4 TPS54560BDDA

Commit message: V1 progress
Parts:
- added U5: CYPD3177-24LQ, Package_DFN_QFN:QFN-24-1EP_4x4mm_P0.5mm_EP2.75x2.75mm, symbol Interface_USB:CYPD3177-24LQ
- C1: footprint (none) -> Capacitor_SMD:C_1206_3216Metric
- J1: footprint (none) -> Connector_USB:USB_C_Receptacle_GCT_USB4135-GF-A_6P_TopMnt_Horizontal
- R11, R12, R13, R14, R15, R16: footprint (none) -> Resistor_SMD:R_1206_3216Metric
Connections:
- new net: U5.19 (GND), U5.22 (GND), U5.25 (GND)
Other:
- note added: "For Cytron RP2040 Motor Controller board bulk capacitance to prevent spikes? GND/PWR screw terminals with 18AWG wire? Connectors? Ensure USB-C connector rated up to 5A"
- note added: "This assembly negotiates required voltage via USB-C PD. Breakout boards for this exist, that could be used in place. Options: 5V (up to 15W) 9V (up to 27W) 15V (up to 45W) 20V (up to 100W) Octopart (ideally DIgikey or Mouser) Connect shield to GND Double check footprint"
- note removed: "For Cytron RP2040 Motor Controller board bulk capacitance to prevent spikes? GND/PWR screw terminals with 18AWG wire? Connectors?"
- note removed: "This assembly negotiates required voltage via USB-C PD. Breakout boards for this exist, that could be used in place. Options: 5V (up to 15W) 9V (up to 27W) 15V (up to 45W) 20V (up to 100W) Octopart (ideally DIgikey or Mouser) Connect shield to GND Double check capacitance allowed by HUSB238"
Changed lines of the file:
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@@
 		)
 	)
-	(text "This assembly negotiates required voltage via USB-C PD. \n\nBreakout boards for this exist, that could be used in place.\n\nOptions: \n5V (up to 15W) \n9V (up to 27W)\n15V (up to 45W)\n20V (up to 100W)\n\nOctopart (ideally DIgikey or Mouser)\nConnect shield to GND\n\nDouble check capacitance allowed by HUSB238"
+	(text "This assembly negotiates required voltage via USB-C PD. \n\nBreakout boards for this exist, that could be used in place.\n\nOptions: \n5V (up to 15W) \n9V (up to 27W)\n15V (up to 45W)\n20V (up to 100W)\n\nOctopart (ideally DIgikey or Mouser)\nConnect shield to GND\n\nDouble check footprint"
 		(exclude_from_sim no)
 		(at 39.624 104.648 0)
@@
 		)
 	)
-	(text "For Cytron RP2040 Motor Controller board\nbulk capacitance to prevent spikes?\nGND/PWR screw terminals with 18AWG wire?\n\nConnectors?"
+	(text "For Cytron RP2040 Motor Controller board\nbulk capacitance to prevent spikes?\nGND/PWR screw terminals with 18AWG wire?\n\nConnectors? \n\nEnsure USB-C connector rated up to 5A"
 		(exclude_from_sim no)
 		(at 352.552 346.202 0)
@@
 	)
 	(symbol
+		(lib_id "Interface_USB:CYPD3177-24LQ")
+		(at 228.6 168.91 0)
+		(unit 1)
+		(body_style 1)
+		(exclude_from_sim no)
+		(in_bom yes)
+		(on_board yes)
+		(in_pos_files yes)
+		(dnp no)
+		(fields_autoplaced yes)
+		(property "Reference" "U5"
+			(at 230.7433 191.77 0)
+			(show_name no)
+			(do_not_autoplace no)
+			(effects
+				(font
+					(size 1.27 1.27)
+				)
+				(justify left)
+			)
+		)
+		(property "Value" "CYPD3177-24LQ"
+			(at 230.7433 194.31 0)
+			(show_name no)
+			(do_not_autoplace no)
+			(effects
+				(font
+					(size 1.27 1.27)
+				)
+				(justify left)
+			)
+		)
+		(property "Footprint" "Package_DFN_QFN:QFN-24-1EP_4x4mm_P0.5mm_EP2.75x2.75mm"
+			(at 228.6 168.91 0)
+			(hide yes)
+			(show_name no)
+			(do_not_autoplace no)
+			(effects
+				(font
+					(size 1.27 1.27)
+				)
+			)
+		)
+		(property "Datasheet" "https://www.infineon.com/dgdl/Infineon-EZ-PD_BCR_Datasheet_USB_Type-C_Port_Controller_for_Power_Sinks-DataSheet-v03_00-EN.pdf?fileId=8ac78c8c7d0d8da4017d0ee7ce9d70ad"
+			(at 228.6 168.91 0)
+			(hide yes)
+			(show_name no)
+			(do_not_autoplace no)
+			(effects
+				(font
+					(size 1.27 1.27)
+				)
+			)
+		)
+		(property "Description" "Stand-alone USB PD controller (with sink Auto-run mode), QFN-24"
+			(at 228.6 168.91 0)
+			(hide yes)
+			(show_name no)
+			(do_not_autoplace no)
+			(effects
+				(font
+					(size 1.27 1.27)
+				)
+			)
+		)
+		(pin "17"
+		)
+		(pin "20"
+		)
+		(pin "18"
+		)
+		(pin "23"
+		)
+		(pin "25"
+		)
+		(pin "19"
+		)
+		(pin "24"
+		)
+		(pin "21"
+		)
+		(pin "22"
+		)
+		(pin "11"
+		)
+		(pin "12"
+		)
+		(pin "13"
+		)
+		(pin "10"
+		)
+		(pin "16"
+		)
+		(pin "15"
+		)
+		(pin "14"
+		)
+		(pin "7"
+		)
+		(pin "1"
+		)
+		(pin "8"
+		)
+		(pin "4"
+		)
+		(pin "9"
+		)
+		(pin "5"
+		)
+		(pin "6"
+		)
+		(pin "2"
+		)
+		(pin "3"
+		)
+		(instances
+			(project "my_power_supply"
+				(path "/08cc4527-d306-41b3-bcbb-e2b853cedcc4"
+					(reference "U5")
+					(unit 1)
+				)
+			)
+		)
+	)
+	(symbol
 		(lib_id "Device:R")
 		(at 121.92 45.72 180)
@@
 			)
 		)
-		(property "Footprint" ""
+		(property "Footprint" "Resistor_SMD:R_1206_3216Metric"
 			(at 135.382 350.52 90)
 			(hide yes)
@@
 			)
 		)
-		(property "Footprint" ""
+		(property "Footprint" "Resistor_SMD:R_1206_3216Metric"
 			(at 126.492 337.82 90)
 			(hide yes)
@@
 			)
 		)
-		(property "Footprint" ""
+		(property "Footprint" "Resistor_SMD:R_1206_3216Metric"
 			(at 219.202 350.52 90)
 			(hide yes)
@@
 			)
 		)
-		(property "Footprint" ""
+		(property "Footprint" "Resistor_SMD:R_1206_3216Metric"
 			(at 219.202 337.82 90)
 			(hide yes)
@@
 			)
 		)
-		(property "Footprint" ""
+		(property "Footprint" "Capacitor_SMD:C_1206_3216Metric"
 			(at 82.2452 53.34 0)
 			(hide yes)
@@
 			)
 		)
-		(property "Footprint" ""
+		(property "Footprint" "Resistor_SMD:R_1206_3216Metric"
 			(at 168.402 345.44 90)
 			(hide yes)
@@
 			)
 		)
-		(property "Footprint" ""
+		(property "Footprint" "Resistor_SMD:R_1206_3216Metric"
 			(at 126.492 350.52 90)
 			(hide yes)
@@
 			)
 		)
-		(property "Footprint" ""
+		(property "Footprint" "Connector_USB:USB_C_Receptacle_GCT_USB4135-GF-A_6P_TopMnt_Horizontal"
 			(at 52.07 60.96 0)
 			(hide yes)

Commit message: Replace HUSB234 with CYPD3177 module
Parts:
- removed C1: 1u, Capacitor_SMD:C_1206_3216Metric, symbol Device:C
- removed J1: USB_C_Receptacle_USB2.0_16P, Connector_USB:USB_C_Receptacle_GCT_USB4135-GF-A_6P_TopMnt_Horizontal, symbol Connector:USB_C_Receptacle_USB2.0_16P
- removed JP1, JP2, JP3, JP4, JP5, JP6, JP7: SolderJumper_2_Open, symbol Jumper:SolderJumper_2_Open
- removed Q1: AONR21307, AONR21307:TRANS_AONR21307, symbol AONR21307:AONR21307
- removed R1: 10, Resistor_SMD:R_1206_3216Metric, symbol Device:R
- removed R2: 5.1k, Resistor_SMD:R_1206_3216Metric, symbol Device:R
- removed R3: 49.9k, Resistor_SMD:R_1206_3216Metric, symbol Device:R
- removed R4, R7: 14k, Resistor_SMD:R_1206_3216Metric, symbol Device:R
- removed R5: 6k, Resistor_SMD:R_1206_3216Metric, symbol Device:R
- removed R6: 10k, Resistor_SMD:R_1206_3216Metric, symbol Device:R
- removed R8: 18k, Resistor_SMD:R_1206_3216Metric, symbol Device:R
- removed U3: HUSB238, HUSB238:DFN-10-1EP_3x3mm_P0.5mm_EP1.65x2.38mm_ThermalVias, symbol HUSB238:HUSB238
- added C2: 3.3u, Capacitor_SMD:C_1206_3216Metric, symbol Device:C
- added C28, C29: 0.1u, Capacitor_SMD:C_1206_3216Metric, symbol Device:C
- added C3, C4: 390p, Capacitor_SMD:C_1206_3216Metric, symbol Device:C
- added C5, C6, C7: 1u, Capacitor_SMD:C_1206_3216Metric, symbol Device:C
- added D1: LED_Small, symbol Device:LED_Small
- added D4: D_Schottky, symbol Device:D_Schottky
- added J4: USB_C_Receptacle_USB2.0_16P, Connector_USB:USB_C_Receptacle_GCT_USB4135-GF-A_6P_TopMnt_Horizontal, symbol Connector:USB_C_Receptacle_USB2.0_16P
- added Q1, Q2: DMP3013SFV, Package_SON:Diodes_PowerDI3333-8, symbol Transistor_FET:DMP3013SFV
- added R23: 2.4k, Resistor_SMD:R_1206_3216Metric, symbol Device:R
- added R24: 47k, Resistor_SMD:R_1206_3216Metric, symbol Device:R
- added R25: 10k, Resistor_SMD:R_1206_3216Metric, symbol Device:R
- added R26: 1k, Resistor_SMD:R_1206_3216Metric, symbol Device:R
Connections:
- net CC1: now also U5.15 (CC1), C3.1, J4.A5 (CC1)
- net CC2: now also U5.14 (CC2), C4.1, J4.B5 (CC2)
- net D+: now also J4.A6 (D+), J4.B6 (D+)
- net D-: now also J4.A7 (D-), J4.B7 (D-)
- net GND: now also U5.1 (VBUS_MIN), U5.19 (GND), U5.22 (GND), U5.25 (GND), U5.6 (ISNK_FINE), C2.2, C28.2, C29.2, C3.2, C4.2, C5.1, C7.2, D1.1 (K), J4.A1 (GND), J4.A12 (GND), J4.B1 (GND), J4.B12 (GND), J4.S1 (SHIELD)
- net VCC: now also Q2.5 (D)
- net VBUSIN: now reaches U5.18 (VBUS_IN)
- net VBUSIN: now also C2.1, C6.1, J4.A4 (VBUS), J4.A9 (VBUS), J4.B4 (VBUS), J4.B9 (VBUS), Q1.5 (D), R25.2
- net 3V3: now reaches U5.2 (VBUS_MAX)
- net 3V3: now also U5.23 (VDDD), U5.5 (ISNK_COARSE), C28.1, C29.1, C7.1
- net at U5.24 (VCCD): now also C5.2
- net at U5.3 (VBUS_FET_EN): now also R26.1
- net at U5.9 (FAULT): now also R23.1
- new net: D1.2 (A), R23.2
- new net: C6.2, D4.2 (A), Q1.4 (G), Q2.4 (G), R24.1, R25.1, R26.2
- new net: D4.1 (K), Q1.1 (S), Q1.2 (S), Q1.3 (S), Q2.1 (S), Q2.2 (S), Q2.3 (S), R24.2
- no-connect marks 8 -> 24
Other:
- note added: "https://github.com/Hugoyhu/CYPD3177-Breakout/blob/main/CYPD3177%20Breakout%20Schematic.png"
- moved on the sheet: SW1, SW2

Commit message: Add footprints for some modules, everything has some kind of footprint to start. Beginning of layout
Parts:
- C10: renamed from C8; footprint (none) -> Capacitor_SMD:C_1206_3216Metric
- C11: renamed from C9; footprint (none) -> Capacitor_SMD:C_1206_3216Metric
- C12: renamed from C10; footprint (none) -> Capacitor_SMD:C_1206_3216Metric
- C13: renamed from C11; footprint (none) -> Capacitor_SMD:C_1206_3216Metric
- C14: renamed from C12; footprint (none) -> Capacitor_SMD:C_1206_3216Metric
- C15: renamed from C13; footprint (none) -> Capacitor_SMD:C_1206_3216Metric
- C16: renamed from C14; footprint (none) -> Capacitor_SMD:C_1206_3216Metric
- C17: renamed from C16; footprint (none) -> Capacitor_SMD:C_1206_3216Metric
- C18: renamed from C15; footprint (none) -> Capacitor_SMD:C_1206_3216Metric
- C19: renamed from C22; footprint (none) -> Capacitor_SMD:C_1206_3216Metric
- C20: renamed from C25; footprint (none) -> Capacitor_SMD:C_1206_3216Metric
- C21: renamed from C26; footprint (none) -> Capacitor_SMD:C_1206_3216Metric
- C22: renamed from C27; footprint (none) -> Capacitor_SMD:C_1206_3216Metric
- C23: renamed from C18; footprint (none) -> Capacitor_SMD:C_1206_3216Metric
- C24: renamed from C19; footprint (none) -> Capacitor_SMD:C_1206_3216Metric
- C25: renamed from C20; footprint (none) -> Capacitor_SMD:C_1206_3216Metric
- C26: renamed from C21; footprint (none) -> Capacitor_SMD:C_1206_3216Metric
- C27: renamed from C24; footprint (none) -> Capacitor_SMD:C_1206_3216Metric
- C28: renamed from C23; footprint (none) -> Capacitor_SMD:C_1206_3216Metric
- C9: renamed from C17; footprint (none) -> Capacitor_SMD:C_1206_3216Metric
- D1: renamed from D4; footprint (none) -> Diode_SMD:D_SOD-323F
- D2: renamed from D1; footprint (none) -> LED_SMD:LED_1206_3216Metric_Pad1.42x1.75mm_HandSolder
- D3: renamed from D2; footprint (none) -> imported:SMC_DIO
- D4: renamed from D3; footprint (none) -> imported:SMC_DIO
- J1: renamed from J4; footprint Connector_USB:USB_C_Receptacle_GCT_USB4135-GF-A_6P_TopMnt_Horizontal -> Connector_USB:USB_C_Plug_Molex_105444
- J2, J3: footprint (none) -> Connector_USB:USB_C_Plug_Molex_105444
- L1: renamed from L2; footprint (none) -> imported:L_Wurth_WE-PDF-1045
- L2: renamed from L3; footprint (none) -> imported:L_Wurth_WE-PDF-1045
- R11: renamed from R17; footprint (none) -> Resistor_SMD:R_1206_3216Metric
- R12: renamed from R21; footprint (none) -> Resistor_SMD:R_1206_3216Metric
- R13: renamed from R20; footprint (none) -> Resistor_SMD:R_1206_3216Metric
- R14: renamed from R18; footprint (none) -> Resistor_SMD:R_1206_3216Metric
- R15: renamed from R19; footprint (none) -> Resistor_SMD:R_1206_3216Metric
- R16: renamed from R22; footprint (none) -> Resistor_SMD:R_1206_3216Metric
- SW1, SW2: footprint (none) -> Button_Switch_SMD:SW_DIP_SPSTx01_Slide_9.78x4.72mm_W8.61mm_P2.54mm
- renumbered C2 to C1, C6 to C2, C7 to C3, C28 to C4, C29 to C5, C3 to C6, C5 to C7, C4 to C8, R25 to R1, R15 to R10, R24 to R2, R26 to R3, R23 to R4, R11 to R5, R16 to R6, R14 to R7, R12 to R8, R13 to R9, U5 to U1, U4 to U3

Commit message: Even more PCB layout
Parts:
- added R17: DNP, Resistor_SMD:R_1206_3216Metric, symbol Device:R
- J1: footprint Connector_USB:USB_C_Plug_Molex_105444 -> Connector_USB:USB_C_Plug_JAE_DX07P024AJ1
Connections:
- net 3V3: now also R17.2
- net GND: now also R17.1
- no-connect marks 24 -> 22
Other:
- note added: "DMP3098 Phil's Lab video https://www.youtube.com/watch?v=W13HNsoHj7A"
- note added: "Replace with 0ohm and DNP"
Changed lines of the file:
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@@
 		)
 	)
+	(text "DMP3098\nPhil's Lab video\nhttps://www.youtube.com/watch?v=W13HNsoHj7A"
+		(exclude_from_sim no)
+		(at 239.522 101.346 0)
+		(effects
+			(font
+				(size 1.27 1.27)
+			)
+		)
+	)
 	(text "For Cytron RP2040 Motor Controller board\nbulk capacitance to prevent spikes?\nGND/PWR screw terminals with 18AWG wire?\n\nConnectors? \n\nEnsure USB-C connector rated up to 5A"
 		(exclude_from_sim no)
@@
 		)
 	)
+	(text "Replace with 0ohm and DNP"
+		(exclude_from_sim no)
+		(at 240.792 227.838 0)
+		(effects
+			(font
+				(size 1.27 1.27)
+			)
+		)
+	)
 	(junction
 		(at 241.3 116.84)
@@
 	)
 	(junction
-		(at 213.36 219.71)
-		(diameter 0)
-		(color 0 0 0 0)
-	)
-	(junction
 		(at 187.96 410.21)
 		(diameter 0)
@@
 	)
 	(junction
+		(at 213.36 219.71)
+		(diameter 0)
+		(color 0 0 0 0)
+	)
+	(junction
 		(at 220.98 391.16)
 		(diameter 0)
@@
 	)
 	(no_connect
-		(at 213.36 229.87)
-	)
-	(no_connect
 		(at 68.58 110.49)
 	)
@@
 	)
 	(no_connect
-		(at 213.36 222.25)
-	)
-	(no_connect
 		(at 50.8 123.19)
 	)
@@
 	(wire
 		(pts
-			(xy 213.36 229.87) (xy 213.36 234.95)
-		)
-		(stroke
-			(width 0)
-			(type default)
-		)
-	)
-	(wire
-		(pts
 			(xy 107.95 415.29) (xy 107.95 421.64)
 		)
@@
 	(wire
 		(pts
+			(xy 213.36 219.71) (xy 213.36 223.52)
+		)
+		(stroke
+			(width 0)
+			(type default)
+		)
+	)
+	(wire
+		(pts
 			(xy 96.52 415.29) (xy 96.52 421.64)
 		)
@@
 	(wire
 		(pts
-			(xy 213.36 219.71) (xy 213.36 222.25)
+			(xy 342.9 135.89) (xy 349.25 135.89)
 		)
 		(stroke
@@
 	(wire
 		(pts
-			(xy 342.9 135.89) (xy 349.25 135.89)
+			(xy 175.26 336.55) (xy 187.96 336.55)
 		)
 		(stroke
@@
 	(wire
 		(pts
-			(xy 175.26 336.55) (xy 187.96 336.55)
+			(xy 162.56 327.66) (xy 166.37 327.66)
 		)
 		(stroke
@@
 	(wire
 		(pts
-			(xy 162.56 327.66) (xy 166.37 327.66)
+			(xy 128.27 417.83) (xy 128.27 420.37)
 		)
 		(stroke
@@
 	(wire
 		(pts
-			(xy 128.27 417.83) (xy 128.27 420.37)
+			(xy 179.07 134.62) (xy 176.53 134.62)
 		)
 		(stroke
@@
 	(wire
 		(pts
-			(xy 179.07 134.62) (xy 176.53 134.62)
+			(xy 213.36 231.14) (xy 213.36 234.95)
 		)
 		(stroke
@@
 	)
 	(symbol
+		(lib_id "Device:R")
+		(at 213.36 227.33 180)
+		(unit 1)
+		(body_style 1)
+		(exclude_from_sim no)
+		(in_bom yes)
+		(on_board yes)
+		(in_pos_files yes)
+		(dnp no)
+		(fields_autoplaced yes)
+		(property "Reference" "R17"
+			(at 215.9 226.0599 0)
+			(show_name no)
+			(do_not_autoplace no)
+			(effects
+				(font
+					(size 1.27 1.27)
+				)
+				(justify right)
+			)
+		)
+		(property "Value" "DNP"
+			(at 215.9 228.5999 0)
+			(show_name no)
+			(do_not_autoplace no)
+			(effects
+				(font
+					(size 1.27 1.27)
+				)
+				(justify right)
+			)
+		)
+		(property "Footprint" "Resistor_SMD:R_1206_3216Metric"
+			(at 215.138 227.33 90)
+			(hide yes)
+			(show_name no)
+			(do_not_autoplace no)
+			(effects
+				(font
+					(size 1.27 1.27)
+				)
+			)
+		)
+		(property "Datasheet" ""
+			(at 213.36 227.33 0)
+			(hide yes)
+			(show_name no)
+			(do_not_autoplace no)
+			(effects
+				(font
+					(size 1.27 1.27)
+				)
+			)
+		)
+		(property "Description" "Resistor"
+			(at 213.36 227.33 0)
+			(hide yes)
+			(show_name no)
+			(do_not_autoplace no)
+			(effects
+				(font
+					(size 1.27 1.27)
+				)
+			)
+		)
+		(pin "2"
+		)
+		(pin "1"
+		)
+		(instances
+			(project "my_power_supply"
+				(path "/08cc4527-d306-41b3-bcbb-e2b853cedcc4"
+					(reference "R17")
+					(unit 1)
+				)
+			)
+		)
+	)
+	(symbol
 		(lib_id "Device:C")
 		(at 198.12 400.05 0)
@@
 			)
 		)
-		(property "Footprint" "Connector_USB:USB_C_Plug_Molex_105444"
+		(property "Footprint" "Connector_USB:USB_C_Plug_JAE_DX07P024AJ1"
 			(at 165.1 132.08 0)
 			(hide yes)

Commit message: Even more more PCB layout
Parts:
- D1: value D_Schottky -> NZH10C
Other:
- moved on the sheet: C6, C8
Changed lines of the file:
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@@
 	)
 	(junction
+		(at 185.42 186.69)
+		(diameter 0)
+		(color 0 0 0 0)
+	)
+	(junction
 		(at 220.98 317.5)
 		(diameter 0)
@@
 	)
 	(junction
-		(at 199.39 166.37)
-		(diameter 0)
-		(color 0 0 0 0)
-	)
-	(junction
 		(at 96.52 347.98)
 		(diameter 0)
@@
 	(wire
 		(pts
+			(xy 186.69 186.69) (xy 185.42 186.69)
+		)
+		(stroke
+			(width 0)
+			(type default)
+		)
+	)
+	(wire
+		(pts
 			(xy 254 194.31) (xy 254 196.85)
 		)
@@
 	(wire
 		(pts
-			(xy 194.31 166.37) (xy 199.39 166.37)
+			(xy 181.61 177.8) (xy 181.61 186.69)
 		)
 		(stroke
@@
 	(wire
 		(pts
-			(xy 194.31 161.29) (xy 199.39 161.29)
+			(xy 186.69 177.8) (xy 186.69 186.69)
 		)
 		(stroke
@@
 	(wire
 		(pts
-			(xy 199.39 161.29) (xy 199.39 166.37)
+			(xy 199.39 161.29) (xy 199.39 168.91)
 		)
 		(stroke
@@
 	(wire
 		(pts
-			(xy 199.39 166.37) (xy 199.39 168.91)
-		)
-		(stroke
-			(width 0)
-			(type default)
-		)
-	)
-	(wire
-		(pts
 			(xy 175.26 391.16) (xy 175.26 396.24)
 		)
@@
 	(wire
 		(pts
-			(xy 181.61 161.29) (xy 186.69 161.29)
+			(xy 186.69 165.1) (xy 186.69 170.18)
 		)
 		(stroke
@@
 	(wire
 		(pts
+			(xy 181.61 186.69) (xy 185.42 186.69)
+		)
+		(stroke
+			(width 0)
+			(type default)
+		)
+	)
+	(wire
+		(pts
 			(xy 156.21 391.16) (xy 137.16 391.16)
 		)
@@
 	(wire
 		(pts
-			(xy 181.61 166.37) (xy 186.69 166.37)
+			(xy 181.61 165.1) (xy 181.61 170.18)
 		)
 		(stroke
@@
 	(global_label "CC2"
 		(shape bidirectional)
-		(at 181.61 166.37 180)
+		(at 181.61 165.1 90)
 		(effects
 			(font
 				(size 1.27 1.27)
 			)
-			(justify right)
+			(justify left)
 		)
 		(property "Intersheetrefs" "${INTERSHEET_REFS}"
-			(at 181.61 166.37 0)
+			(at 181.61 165.1 90)
 			(hide yes)
 			(show_name no)
@@
 	(global_label "CC1"
 		(shape bidirectional)
-		(at 181.61 161.29 180)
+		(at 186.69 165.1 90)
 		(effects
 			(font
 				(size 1.27 1.27)
 			)
-			(justify right)
+			(justify left)
 		)
 		(property "Intersheetrefs" "${INTERSHEET_REFS}"
-			(at 181.61 161.29 0)
+			(at 186.69 165.1 90)
 			(hide yes)
 			(show_name no)
@@
 	(symbol
 		(lib_id "power:GND")
-		(at 199.39 168.91 0)
+		(at 185.42 186.69 0)
 		(unit 1)
 		(body_style 1)
@@
 		(fields_autoplaced yes)
 		(property "Reference" "#PWR04"
-			(at 199.39 175.26 0)
+			(at 185.42 193.04 0)
 			(hide yes)
 			(show_name no)
@@
 		)
 		(property "Value" "GND"
-			(at 199.39 173.99 0)
+			(at 187.96 187.9599 0)
 			(show_name no)
 			(do_not_autoplace no)
@@
 					(size 1.27 1.27)
 				)
+				(justify left)
 			)
 		)
 		(property "Footprint" ""
-			(at 199.39 168.91 0)
+			(at 185.42 186.69 0)
 			(hide yes)
 			(show_name no)
@@
 		)
 		(property "Datasheet" ""
-			(at 199.39 168.91 0)
+			(at 185.42 186.69 0)
 			(hide yes)
 			(show_name no)
@@
 		)
 		(property "Description" "Power symbol creates a global label with name \"GND\" , ground"
-			(at 199.39 168.91 0)
+			(at 185.42 186.69 0)
 			(hide yes)
 			(show_name no)
@@
 	(symbol
 		(lib_id "Device:C")
-		(at 190.5 166.37 90)
+		(at 181.61 173.99 0)
 		(unit 1)
 		(body_style 1)
@@
 		(dnp no)
 		(property "Reference" "C8"
-			(at 190.246 170.18 90)
+			(at 177.8 173.736 90)
 			(show_name no)
 			(do_not_autoplace no)
@@
 		)
 		(property "Value" "390p"
-			(at 190.5 172.212 90)
+			(at 175.768 173.99 90)
 			(show_name no)
 			(do_not_autoplace no)
@@
 		)
 		(property "Footprint" "Capacitor_SMD:C_1206_3216Metric"
-			(at 194.31 165.4048 0)
+			(at 182.5752 177.8 0)
 			(hide yes)
 			(show_name no)
@@
 		)
 		(property "Datasheet" ""
-			(at 190.5 166.37 0)
+			(at 181.61 173.99 0)
 			(hide yes)
 			(show_name no)
@@
 		)
 		(property "Description" "Unpolarized capacitor"
-			(at 190.5 166.37 0)
+			(at 181.61 173.99 0)
 			(hide yes)
 			(show_name no)
@@
 	(symbol
 		(lib_id "Device:C")
-		(at 190.5 161.29 90)
+		(at 186.69 173.99 0)
 		(unit 1)
 		(body_style 1)
@@
 		(dnp no)
 		(property "Reference" "C6"
-			(at 190.5 155.448 90)
+			(at 192.532 173.99 90)
 			(show_name no)
 			(do_not_autoplace no)
@@
 		)
 		(property "Value" "390p"
-			(at 190.754 157.48 90)
+			(at 190.5 174.244 90)
 			(show_name no)
 			(do_not_autoplace no)
@@
 		)
 		(property "Footprint" "Capacitor_SMD:C_1206_3216Metric"
-			(at 194.31 160.3248 0)
+			(at 187.6552 177.8 0)
 			(hide yes)
 			(show_name no)
@@
 		)
 		(property "Datasheet" ""
-			(at 190.5 161.29 0)
+			(at 186.69 173.99 0)
 			(hide yes)
 			(show_name no)
@@
 		)
 		(property "Description" "Unpolarized capacitor"
-			(at 190.5 161.29 0)
+			(at 186.69 173.99 0)
 			(hide yes)
 			(show_name no)
@@
 			)
 		)
-		(property "Value" "D_Schottky"
+		(property "Value" "NZH10C"
 			(at 228.6 125.4124 90)
 			(show_name no)
